File: 19__Loadcell_Module_ HX711.kicad_sch (KiCad schematic)
At the start: 16 parts, among them J1 Screw_Terminal_01x06, Q1 MMBT3906, U1 HX711

Commit message: Add files via upload
Parts:
- added D1: LED, LED_SMD:LED_0805_2012Metric, symbol Device:LED
- added R7: 470r, Resistor_SMD:R_0805_2012Metric, symbol Device:R
- added U2: ~, Moduler_:pin_header, symbol moduler_pin:air
- C1, C2, C3, C4, C5, C6, C7: footprint (none) -> Capacitor_SMD:C_0805_2012Metric
- J1: footprint (none) -> TerminalBlock_Phoenix:TerminalBlock_Phoenix_PT-1,5-6-3.5-H_1x06_P3.50mm_Horizontal
- R1, R2, R3, R4, R5, R6: footprint (none) -> Resistor_SMD:R_0805_2012Metric
Connections:
- net VCC is gone; now on net +5V: C6.1, C7.1, U1.16 (DVDD)
- net CLK: now also U2.12
- net DOUT: now also U2.13
- net GND: now also D1.1 (K), U2.9
- net RATE: now also U2.3
- net +5V: now reaches Q1.2 (E), U1.1 (VSUP)
- net +5V: now also R7.1, U2.7
- new net: D1.2 (A), R7.2
- no-connect marks 1 -> 14
Other:
- note added: "AIR PIN"
- note added: "LOAD CHANNEL"
- note added: "SENSOR"
- moved on the sheet: C1, C2, C3, C4, C5, C6, C7, J1, Q1, R1, R2, R3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
